File: kicad/ESP32-MUSEU/ESP32-MUSEU.sch (KiCad schematic (older format))
At the start: 8 parts

Commit message: Finished wiring as in the mounted pcb
Parts:
- gave numbers to parts that had none: 8
Connections:
- net LDR: now also U1.5 (D4)
- net TX2: now reaches A1.4 (RXD)
- net TX2: now also U1.7 (TX2)
- net RX2: now reaches A1.5 (TXD)
- net RX2: now also U1.6 (RX2)
- net TXS: now reaches U1.24 (D26)
- net TXS: now also A5.8 (UART_RxD)
- net CAL: now reaches U1.25 (D27)
- net CAL: now also A5.5 (bCAL_in)
- net RXS: now reaches U1.28 (D13)
- net RXS: now also A5.7 (UART_TxD)
- no-connect marks 7 -> 21
Changed lines of the file:
@@
 $EndDescr
 $Comp
-L esp32_devkit_v1:ESP32_DEVKIT_V1 U?
-U 1 1 5FB13BB6
-P 5300 2000
-F 0 "U?" H 5300 3215 50  0000 C CNN
-F 1 "ESP32_DEVKIT_V1" H 5300 3124 50  0000 C CNN
-F 2 "" H 5300 2100 50  0001 C CNN
-F 3 "" H 5300 2100 50  0001 C CNN
-	1    5300 2000
-	1    0    0    -1
-$EndComp
-$Comp
-L igorkelvin:SDCard_Module A?
+L igorkelvin:SDCard_Module A4
 U 1 1 5FB19464
 P 7500 3500
-F 0 "A?" H 8128 3596 50  0000 L CNN
+F 0 "A4" H 8128 3596 50  0000 L CNN
 F 1 "SDCard_Module" H 8128 3505 50  0000 L CNN
 F 2 "" H 7450 4200 50  0001 C CNN
@@
 $EndComp
 $Comp
-L igorkelvin:DS3231_Module A?
+L igorkelvin:DS3231_Module A3
 U 1 1 5FB1770C
 P 7500 2500
-F 0 "A?" H 8078 2601 50  0000 L CNN
+F 0 "A3" H 8078 2601 50  0000 L CNN
 F 1 "DS3231_Module" H 8078 2510 50  0000 L CNN
 F 2 "" H 6500 2700 50  0001 C CNN
@@
 	6900 1400 7000 1400
 $Comp
-L senseair_s8_module:SenseAir_S8_Module A?
+L senseair_s8_module:SenseAir_S8_Module A5
 U 1 1 5FB1BDE1
 P 7600 1500
-F 0 "A?" H 7600 1965 50  0000 C CNN
+F 0 "A5" H 7600 1965 50  0000 C CNN
 F 1 "SenseAir_S8_Module" H 7600 1874 50  0000 C CNN
 F 2 "" H 7600 1400 50  0001 C CNN
@@
 	4000 3100 3900 3100
 $Comp
-L winsen_zh06_module:Winsen_ZH06_Module A?
+L winsen_zh06_module:Winsen_ZH06_Module A1
 U 1 1 5FB091C1
 P 3300 3400
-F 0 "A?" H 3828 3496 50  0000 L CNN
+F 0 "A1" H 3828 3496 50  0000 L CNN
 F 1 "Winsen_ZH06_Module" H 3828 3405 50  0000 L CNN
 F 2 "" H 3300 4000 50  0001 C CNN
@@
 3V3
 $Comp
-L bme280_module:BME280_Module A?
+L bme280_module:BME280_Module A2
 U 1 1 5FB154D9
 P 3450 1450
-F 0 "A?" H 3728 1501 50  0000 L CNN
+F 0 "A2" H 3728 1501 50  0000 L CNN
 F 1 "BME280_Module" H 3728 1410 50  0000 L CNN
 F 2 "" H 3400 1400 50  0001 C CNN
@@
 $EndComp
 $Comp
-L Device:R_US R?
+L Device:R_US R2
 U 1 1 5FB92941
 P 3300 2350
-F 0 "R?" H 3368 2396 50  0000 L CNN
+F 0 "R2" H 3368 2396 50  0000 L CNN
 F 1 "10K" H 3368 2305 50  0000 L CNN
 F 2 "" V 3340 2340 50  0001 C CNN
@@
 	1400 1500 1400 1800
 $Comp
-L power:GNDREF #PWR?
+L power:GNDREF #PWR02
 U 1 1 5FBA23F0
 P 1400 1800
-F 0 "#PWR?" H 1400 1550 50  0001 C CNN
+F 0 "#PWR02" H 1400 1550 50  0001 C CNN
 F 1 "GNDREF" H 1405 1627 50  0000 C CNN
 F 2 "" H 1400 1800 50  0001 C CNN
@@
 $EndComp
 $Comp
-L power:+5V #PWR?
+L power:+5V #PWR03
 U 1 1 5FBA2BB8
 P 1700 1200
-F 0 "#PWR?" H 1700 1050 50  0001 C CNN
+F 0 "#PWR03" H 1700 1050 50  0001 C CNN
 F 1 "+5V" H 1715 1373 50  0000 C CNN
 F 2 "" H 1700 1200 50  0001 C CNN
@@
 $EndComp
 $Comp
-L power:+3V3 #PWR?
+L power:+3V3 #PWR01
 U 1 1 5FBA337C
 P 1400 1200
-F 0 "#PWR?" H 1400 1050 50  0001 C CNN
+F 0 "#PWR01" H 1400 1050 50  0001 C CNN
 F 1 "+3V3" H 1415 1373 50  0000 C CNN
 F 2 "" H 1400 1200 50  0001 C CNN
@@
 	1300 1400 1400 1400
 $Comp
-L power:GNDREF #PWR?
+L power:GNDREF #PWR04
 U 1 1 5FBB86D6
 P 3300 2600
-F 0 "#PWR?" H 3300 2350 50  0001 C CNN
+F 0 "#PWR04" H 3300 2350 50  0001 C CNN
 F 1 "GNDREF" H 3305 2427 50  0000 C CNN
 F 2 "" H 3300 2600 50  0001 C CNN
@@
 	3300 2200 3300 2100
 $Comp
-L Device:R_PHOTO R?
+L Device:R_PHOTO R1
 U 1 1 5FB14BF4
 P 3050 2100
-F 0 "R?" H 3120 2146 50  0000 L CNN
+F 0 "R1" H 3120 2146 50  0000 L CNN
 F 1 "R_PHOTO" H 3120 2055 50  0000 L CNN
 F 2 "" V 3100 1850 50  0001 L CNN
@@
 Wire Wire Line
 	4500 2000 4600 2000
+Text Label 4500 1700 2    50   ~ 0
+LDR
+Wire Wire Line
+	4500 1700 4600 1700
+Text Label 4000 3300 0    50   ~ 0
+TX2
+Text Label 4500 1900 2    50   ~ 0
+TX2
+Wire Wire Line
+	4500 1900 4600 1900
+Wire Wire Line
+	4000 3300 3900 3300
+Text Label 4000 3400 0    50   ~ 0
+RX2
+Wire Wire Line
+	4000 3400 3900 3400
+Text Label 4500 1800 2    50   ~ 0
+RX2
+Wire Wire Line
+	4500 1800 4600 1800
+Text Label 6100 1500 0    50   ~ 0
+RXS
+Wire Wire Line
+	6100 1500 6000 1500
+Text Label 8300 1500 0    50   ~ 0
+RXS
+Wire Wire Line
+	8300 1500 8200 1500
+Text Label 6100 1900 0    50   ~ 0
+TXS
+Wire Wire Line
+	6100 1900 6000 1900
+Text Label 8300 1400 0    50   ~ 0
+TXS
+Wire Wire Line
+	8200 1400 8300 1400
+Text Label 6100 1800 0    50   ~ 0
+CAL
+Wire Wire Line
+	6100 1800 6000 1800
+Text Label 8300 1700 0    50   ~ 0
+CAL
+Wire Wire Line
+	8300 1700 8200 1700
+$Comp
+L esp32_devkit_v1:ESP32_DEVKIT_V1 U1
+U 1 1 5FB13BB6
+P 5300 2000
+F 0 "U1" H 5300 3215 50  0000 C CNN
+F 1 "ESP32_DEVKIT_V1" H 5300 3124 50  0000 C CNN
+F 2 "" H 5300 2100 50  0001 C CNN
+F 3 "" H 5300 2100 50  0001 C CNN
+	1    5300 2000
+	1    0    0    -1
+$EndComp
+NoConn ~ 4600 1500
+NoConn ~ 4600 1600
+NoConn ~ 4600 2400
+NoConn ~ 4600 2500
+NoConn ~ 6000 2700
+NoConn ~ 6000 2600
+NoConn ~ 6000 2500
+NoConn ~ 6000 2400
+NoConn ~ 6000 2300
+NoConn ~ 6000 2200
+NoConn ~ 6000 2100
+NoConn ~ 6000 2000
+NoConn ~ 6000 1700
+NoConn ~ 6000 1600
 $EndSCHEMATC
