File: kicad/ESP32-MUSEU.sch (KiCad schematic (older format))
At the start: 8 parts, among them U1 ESP32_DEVKIT_V1

Commit message: Included external reset pushbutton
Parts:
- added SW1: SW_Push, symbol Switch:SW_Push
Connections:
- net GNDREF: now also SW1.1
- net LDR: now also U1.19 (D34); no longer U1.22 (D33)
- net EN: now reaches U1.16 (EN)
- net EN: now also SW1.2
- no-connect marks 21 -> 20
Changed lines of the file:
@@
 Wire Wire Line
 	4500 2000 4600 2000
-Text Label 6100 2100 0    50   ~ 0
+Text Label 6100 2400 0    50   ~ 0
 LDR
 Text Label 4000 3300 0    50   ~ 0
@@
 NoConn ~ 4600 2400
 NoConn ~ 4600 2500
-NoConn ~ 6000 2700
 NoConn ~ 6000 2600
 NoConn ~ 6000 2500
-NoConn ~ 6000 2400
 NoConn ~ 6000 2300
 NoConn ~ 6000 2200
@@
 NoConn ~ 6000 1600
 Wire Wire Line
-	6000 2100 6100 2100
+	6000 2400 6100 2400
 NoConn ~ 4600 1700
+NoConn ~ 6000 2100
+$Comp
+L Switch:SW_Push SW1
+U 1 1 5FB403F5
+P 5300 3600
+F 0 "SW1" H 5300 3885 50  0000 C CNN
+F 1 "SW_Push" H 5300 3794 50  0000 C CNN
+F 2 "" H 5300 3800 50  0001 C CNN
+F 3 "~" H 5300 3800 50  0001 C CNN
+	1    5300 3600
+	1    0    0    -1
+$EndComp
+Text Label 5000 3600 2    50   ~ 0
+GND
+Text Label 5600 3600 0    50   ~ 0
+EN
+Text Label 6100 2700 0    50   ~ 0
+EN
+Wire Wire Line
+	5600 3600 5500 3600
+Wire Wire Line
+	5100 3600 5000 3600
+Wire Wire Line
+	6100 2700 6000 2700
 $EndSCHEMATC

Commit message: Updated led pins, Added R3 and updated LDR name
Parts:
- added D1: LED_RGBA, symbol Device:LED_RGBA
- added R3: 940Ω, symbol Device:R_US
- R1: value R_PHOTO -> GL10528
- R2: value 10K -> 10KΩ
Connections:
- net +3V3: now also R3.1
- net LED_B: now reaches U1.13 (TX0)
- net LED_B: now also D1.3 (BK)
- net LED_R: now reaches U1.22 (D33)
- net LED_R: now also D1.1 (RK)
- new net: D1.4 (A), R3.2
- no-connect marks 20 -> 19
Changed lines of the file:
@@
 P 3300 2350
 F 0 "R2" H 3368 2396 50  0000 L CNN
-F 1 "10K" H 3368 2305 50  0000 L CNN
+F 1 "10KΩ" H 3368 2305 50  0000 L CNN
 F 2 "" V 3340 2340 50  0001 C CNN
 F 3 "~" H 3300 2350 50  0001 C CNN
@@
 U 1 1 5FB14BF4
 P 3050 2100
-F 0 "R1" H 3120 2146 50  0000 L CNN
-F 1 "R_PHOTO" H 3120 2055 50  0000 L CNN
+F 0 "R1" V 3250 2050 50  0000 L CNN
+F 1 "GL10528" V 3150 1950 50  0000 L CNN
 F 2 "" V 3100 1850 50  0001 L CNN
 F 3 "~" H 3050 2050 50  0001 C CNN
@@
 NoConn ~ 4600 1600
 NoConn ~ 4600 2400
-NoConn ~ 4600 2500
 NoConn ~ 6000 2600
 NoConn ~ 6000 2500
 NoConn ~ 6000 2300
-NoConn ~ 6000 2200
-NoConn ~ 6000 2000
-NoConn ~ 6000 1700
-NoConn ~ 6000 1600
 Wire Wire Line
 	6000 2400 6100 2400
 NoConn ~ 4600 1700
-NoConn ~ 6000 2100
 $Comp
 L Switch:SW_Push SW1
@@
 Wire Wire Line
 	6100 2700 6000 2700
+$Comp
+L Device:LED_RGBA D1
+U 1 1 5FB44AAD
+P 5200 4400
+F 0 "D1" H 5200 4897 50  0000 C CNN
+F 1 "LED_RGBA" H 5200 4806 50  0000 C CNN
+F 2 "" H 5200 4350 50  0001 C CNN
+F 3 "~" H 5200 4350 50  0001 C CNN
+	1    5200 4400
+	1    0    0    -1
+$EndComp
+Text Label 5900 4400 0    50   ~ 0
+3V3
+Wire Wire Line
+	5500 4400 5400 4400
+Text Label 4900 4200 2    50   ~ 0
+LED_R
+Wire Wire Line
+	5000 4600 4900 4600
+Wire Wire Line
+	5000 4400 4900 4400
+Wire Wire Line
+	5000 4200 4900 4200
+Text Label 6100 2100 0    50   ~ 0
+LED_R
+Text Label 4500 2500 2    50   ~ 0
+LED_B
+Wire Wire Line
+	6100 2100 6000 2100
+Wire Wire Line
+	4500 2500 4600 2500
+NoConn ~ 6000 2200
+NoConn ~ 6000 2000
+$Comp
+L Device:R_US R3
+U 1 1 5FB849EF
+P 5650 4400
+F 0 "R3" V 5550 4350 50  0000 L CNN
+F 1 "940Ω" V 5750 4350 50  0000 L CNN
+F 2 "" V 5690 4390 50  0001 C CNN
+F 3 "~" H 5650 4400 50  0001 C CNN
+	1    5650 4400
+	0    1    1    0
+$EndComp
+Wire Wire Line
+	5900 4400 5800 4400
+Text Label 4900 4600 2    50   ~ 0
+LED_B
+NoConn ~ 4900 4400
+NoConn ~ 6000 1700
+NoConn ~ 6000 1600
 $EndSCHEMATC
